File: SAME54-board/SAME54-board.brd (EAGLE design)
At the start: 70.8 x 119.4 mm, 32 parts, among them IC1 ATSAME54N20A-AUT, J1 GSD09002SEU, J2 CON-SOCJ-2155

Commit message: Added drill holes and correct power supply mistake
Parts:
- added R10: 1k, rcl:M1206
- moved C8 1.27 mm to (20.3, 41.9)
Connections:
- net SWDCLK: now also R10.1
- net VCC: now also R10.2
- net VDDIO: now also C5.1, FL1.1, FL1.2, FL1.3, FL1.4
- net VDDIOB: no longer C5.1, FL1.1, FL1.2, FL1.3, FL1.4
Routing:
- net VDDIO: track 50.6 -> 116.9 mm, vias 2 -> 4
- net VCC: track 5.35 -> 15.8 mm, vias 2 -> 4
- net VDDIOB: track 111.6 -> 103.8 mm
- net SWDCLK: track 122.4 -> 128.1 mm
- net VDDANA: track 108.9 -> 110.0 mm
- net GND: track 70.7 -> 71.2 mm
Changed lines of the file:
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@@
 <grid distance="50" unitdist="mil" unit="mil" style="lines" multiple="1" display="no" altdistance="5" altunitdist="mil" altunit="mil"/>
 <layers>
-<layer number="1" name="Top" color="4" fill="1" visible="no" active="yes"/>
-<layer number="16" name="Bottom" color="1" fill="1" visible="no" active="yes"/>
+<layer number="1" name="Top" color="4" fill="1" visible="yes" active="yes"/>
+<layer number="16" name="Bottom" color="1" fill="1" visible="yes" active="yes"/>
 <layer number="17" name="Pads" color="2" fill="1" visible="yes" active="yes"/>
 <layer number="18" name="Vias" color="2" fill="1" visible="yes" active="yes"/>
@@
 PA22
 PA21</text>
+<hole x="1.27" y="1.27" drill="1"/>
+<hole x="69.85" y="1.27" drill="1"/>
+<hole x="1.27" y="118.11" drill="1"/>
+<hole x="69.85" y="118.11" drill="1"/>
 </plain>
 <attributes>
@@
 <attribute name="VALUE" x="43.18" y="67.31" size="1.27" layer="27"/>
 </element>
-<element name="C8" library="rcl" library_urn="urn:adsk.eagle:library:334" package="C1206" package3d_urn="urn:adsk.eagle:package:23618/2" value="100n" x="19.05" y="41.91" smashed="yes" rot="R270">
-<attribute name="NAME" x="20.32" y="40.64" size="1.27" layer="25"/>
-<attribute name="POPULARITY" value="54" x="-41.91" y="-25.4" size="1.778" layer="27" rot="R270" display="off"/>
-<attribute name="SPICEPREFIX" value="C" x="-41.91" y="-25.4" size="1.778" layer="27" rot="R270" display="off"/>
-<attribute name="VALUE" x="16.51" y="43.18" size="1.27" layer="27" rot="R270"/>
+<element name="C8" library="rcl" library_urn="urn:adsk.eagle:library:334" package="C1206" package3d_urn="urn:adsk.eagle:package:23618/2" value="100n" x="20.32" y="41.91" smashed="yes" rot="R270">
+<attribute name="NAME" x="21.59" y="40.64" size="1.27" layer="25"/>
+<attribute name="POPULARITY" value="54" x="-40.64" y="-25.4" size="1.778" layer="27" rot="R270" display="off"/>
+<attribute name="SPICEPREFIX" value="C" x="-40.64" y="-25.4" size="1.778" layer="27" rot="R270" display="off"/>
+<attribute name="VALUE" x="17.78" y="43.18" size="1.27" layer="27" rot="R270"/>
 </element>
 <element name="C9" library="rcl" library_urn="urn:adsk.eagle:library:334" package="C1206" package3d_urn="urn:adsk.eagle:package:23618/2" value="100n" x="29.21" y="38.1" smashed="yes" rot="R180">
@@
 <attribute name="NAME" x="5.08" y="102.87" size="1.27" layer="25" rot="R90" align="center"/>
 </element>
+<element name="R10" library="rcl" library_urn="urn:adsk.eagle:library:334" package="M1206" package3d_urn="urn:adsk.eagle:package:23566/2" value="1k" x="16.51" y="41.91" smashed="yes" rot="R270">
+<attribute name="NAME" x="17.78" y="43.18" size="1.27" layer="25" rot="R270"/>
+<attribute name="POPULARITY" value="22" x="16.51" y="41.91" size="1.778" layer="27" rot="R270" display="off"/>
+<attribute name="SPICEPREFIX" value="R" x="16.51" y="41.91" size="1.778" layer="27" rot="R270" display="off"/>
+<attribute name="VALUE" x="13.97" y="43.18" size="1.27" layer="27" rot="R270"/>
+</element>
 </elements>
 <signals>
 <signal name="VDDIOB">
 <wire x1="27.822" y1="44.8" x2="31.56" y2="44.8" width="0.3048" layer="1"/>
-<contactref element="FL1" pad="1"/>
-<contactref element="FL1" pad="2"/>
-<contactref element="FL1" pad="3"/>
-<contactref element="FL1" pad="4"/>
 <wire x1="31.56" y1="43.062" x2="31.56" y2="44.8" width="0.3048" layer="1"/>
 <wire x1="31.56" y1="44.8" x2="31.56" y2="46.26086875" width="0.3048" layer="1"/>
 <wire x1="31.56" y1="46.26086875" x2="35.377" y2="46.26086875" width="0.3048" layer="1"/>
 <via x="35.377" y="46.26086875" extent="1-16" drill="0.35"/>
-<wire x1="50.33" y1="92.64" x2="50.33" y2="91.84" width="0.2032" layer="1"/>
-<wire x1="50.33" y1="91.84" x2="50.33" y2="91.04" width="0.2032" layer="1"/>
-<wire x1="50.33" y1="91.04" x2="50.33" y2="90.24" width="0.2032" layer="1"/>
 <wire x1="55.75" y1="92.71" x2="55.75" y2="92.64" width="0.2032" layer="1"/>
-<wire x1="55.75" y1="92.64" x2="50.33" y2="92.64" width="0.2032" layer="1"/>
 <wire x1="57.15" y1="88.9" x2="57.15" y2="90.17" width="0.3048" layer="16"/>
 <via x="57.15" y="90.17" extent="1-16" drill="0.35"/>
-<wire x1="57.15" y1="90.17" x2="55.75" y2="90.17" width="0.3048" layer="1"/>
 <wire x1="60.198" y1="88.9" x2="57.15" y2="88.9" width="0.3048" layer="16"/>
-<wire x1="55.75" y1="92.71" x2="55.88" y2="92.71" width="0.3048" layer="1"/>
-<wire x1="55.75" y1="90.17" x2="55.75" y2="92.71" width="0.3048" layer="1"/>
+<wire x1="55.88" y1="92.71" x2="55.75" y2="92.71" width="0.3048" layer="1"/>
 <wire x1="35.377" y1="46.26086875" x2="60.198" y2="46.26086875" width="0.3048" layer="16"/>
 <wire x1="60.198" y1="46.26086875" x2="60.198" y2="69.85" width="0.3048" layer="16"/>
@@
 <contactref element="IC1" pad="30"/>
 <contactref element="C7" pad="1"/>
-<contactref element="C5" pad="1"/>
 <contactref element="C4" pad="1"/>
+<wire x1="57.15" y1="90.17" x2="56.804" y2="90.17" width="0.2032" layer="1"/>
+<wire x1="56.804" y1="90.17" x2="56.804" y2="91.324" width="0.2032" layer="1"/>
+<wire x1="56.804" y1="91.324" x2="55.75" y2="91.324" width="0.2032" layer="1"/>
+<wire x1="55.75" y1="91.324" x2="55.75" y2="92.71" width="0.2032" layer="1"/>
 </signal>
 <signal name="VDDIO">
-<wire x1="30.61" y1="38.1" x2="33.9278" y2="38.1" width="0.2032" layer="1"/>
 <via x="33.9278" y="38.1" extent="1-16" drill="0.35"/>
 <wire x1="35.56" y1="38.1" x2="33.9278" y2="38.1" width="0.2032" layer="16"/>
@@
 <contactref element="IC1" pad="77"/>
 <contactref element="IC1" pad="92"/>
+<contactref element="FL1" pad="1"/>
+<contactref element="FL1" pad="2"/>
+<contactref element="FL1" pad="3"/>
+<contactref element="FL1" pad="4"/>
+<contactref element="C5" pad="1"/>
 <contactref element="C9" pad="1"/>
+<wire x1="50.33" y1="92.64" x2="50.33" y2="91.84" width="0.2032" layer="1"/>
+<wire x1="50.33" y1="91.84" x2="50.33" y2="91.04" width="0.2032" layer="1"/>
+<wire x1="50.33" y1="91.04" x2="50.33" y2="90.24" width="0.2032" layer="1"/>
+<wire x1="30.61" y1="38.1" x2="32.2862" y2="38.1" width="0.2032" layer="1"/>
+<wire x1="32.2862" y1="38.1" x2="32.2862" y2="37.9984" width="0.2032" layer="1"/>
+<wire x1="32.2862" y1="37.9984" x2="33.7538" y2="37.9984" width="0.2032" layer="1"/>
+<wire x1="33.7538" y1="37.9984" x2="33.7538" y2="38.1" width="0.2032" layer="1"/>
+<wire x1="33.7538" y1="38.1" x2="33.9278" y2="38.1" width="0.2032" layer="1"/>
+<wire x1="50.33" y1="90.24" x2="55.75" y2="90.24" width="0.2032" layer="1"/>
+<wire x1="55.75" y1="90.24" x2="55.75" y2="90.17" width="0.2032" layer="1"/>
+<wire x1="50.33" y1="90.24" x2="50.33" y2="88.9" width="0.2032" layer="1"/>
+<wire x1="50.33" y1="88.9" x2="50.8" y2="88.9" width="0.2032" layer="1"/>
+<via x="50.8" y="88.9" extent="1-16" drill="0.35"/>
+<wire x1="50.8" y1="88.9" x2="50.8" y2="88.138" width="0.2032" layer="16"/>
+<wire x1="50.8" y1="88.138" x2="58.928" y2="88.138" width="0.2032" layer="16"/>
+<wire x1="58.928" y1="88.138" x2="58.928" y2="74.422" width="0.2032" layer="16"/>
+<wire x1="41.0962" y1="74.422" x2="41.0962" y2="60.96" width="0.2032" layer="16"/>
+<via x="41.0962" y="60.96" extent="1-16" drill="0.35"/>
+<wire x1="41.0962" y1="60.96" x2="41.0962" y2="58.538" width="0.2032" layer="1"/>
+<wire x1="41.0962" y1="58.538" x2="41.06" y2="58.538" width="0.2032" layer="1"/>
+<wire x1="58.928" y1="74.422" x2="41.0962" y2="74.422" width="0.2032" layer="16"/>
 </signal>
 <signal name="VDDANA">
@@
 <contactref element="FL1" pad="6"/>
 <contactref element="FL1" pad="5"/>
-<wire x1="19.05" y1="43.31" x2="19.05" y2="43.18" width="0.3048" layer="1"/>
+<wire x1="20.32" y1="43.31" x2="20.32" y2="41.91" width="0.3048" layer="1"/>
 <via x="19.05" y="51.4322" extent="1-16" drill="0.35"/>
 <wire x1="19.05" y1="51.4322" x2="19.05" y2="51.3" width="0.3048" layer="1"/>
@@
 <wire x1="43.18" y1="89.662" x2="11.43" y2="89.662" width="0.3048" layer="16"/>
 <wire x1="11.43" y1="89.662" x2="11.43" y2="51.4322" width="0.3048" layer="16"/>
-<wire x1="19.05" y1="43.31" x2="19.05" y2="41.91" width="0.3048" layer="1"/>
-<via x="19.05" y="41.91" extent="1-16" drill="0.35"/>
-<wire x1="19.05" y1="41.91" x2="19.05" y2="51.4322" width="0.3048" layer="16"/>
+<via x="20.32" y="41.91" extent="1-16" drill="0.35"/>
 <contactref element="IC1" pad="12"/>
 <contactref element="C6" pad="1"/>
 <contactref element="C8" pad="1"/>
+<wire x1="19.05" y1="51.4322" x2="19.05" y2="41.91" width="0.3048" layer="16"/>
+<wire x1="19.05" y1="41.91" x2="20.32" y2="41.91" width="0.3048" layer="16"/>
 </signal>
 <signal name="VSW">
@@
 <wire x1="17.78" y1="75.000190625" x2="19.120190625" y2="75.000190625" width="0.2032" layer="16"/>
 <via x="19.120190625" y="75.000190625" extent="1-16" drill="0.35"/>
+<contactref element="R10" pad="2"/>
+<wire x1="16.51" y1="40.51" x2="16.51" y2="35.56" width="0.2032" layer="1"/>
+<wire x1="16.51" y1="35.56" x2="17.78" y2="35.56" width="0.2032" layer="1"/>
+<via x="17.78" y="35.56" extent="1-16" drill="0.35"/>
+<wire x1="17.78" y1="35.56" x2="17.78" y2="31.321" width="0.2032" layer="16"/>
+<via x="17.78" y="31.321" extent="1-16" drill="0.35"/>
 </signal>
 <signal name="RESETN">
@@
 <contactref element="TRACE" pad="17"/>
 <contactref element="CORTEX" pad="7"/>
+<contactref element="R10" pad="1"/>
+<wire x1="20.32" y1="45.1678" x2="16.51" y2="45.1678" width="0.2032" layer="1"/>
+<wire x1="16.51" y1="45.1678" x2="16.51" y2="43.31" width="0.2032" layer="1"/>
 </signal>
 <signal name="SWDIO">
@@
 <via x="57.15" y="92.71" extent="1-16" drill="0.35"/>
 <wire x1="27.81" y1="38.1" x2="19.05" y2="38.1" width="0.2032" layer="1"/>
-<wire x1="19.05" y1="38.1" x2="19.05" y2="40.51" width="0.2032" layer="1"/>
+<wire x1="19.05" y1="38.1" x2="20.32" y2="39.37" width="0.2032" layer="1"/>
+<wire x1="20.32" y1="40.51" x2="20.32" y2="39.37" width="0.2032" layer="1"/>
 <via x="19.05" y="38.1" extent="1-16" drill="0.35"/>
 <wire x1="30.63" y1="30.693" x2="31.426" y2="30.693" width="0.2032" layer="1"/>
