File: board_design/SAME54-board1.0.2.sch (EAGLE design)
At the start: 32 parts, among them IC1 ATSAME54N20A-AUT, J1 PJ-070BH-SMT-TR, M1 NVMFS5C468NL, M2 NVMFS5C468NL, M3 NVMFS5C468NL, M4 NVMFS5C468NL, U1 MAX20034ATIS/VY+

Commit message: Added power and max20034 to schematic
Parts:
- removed CBIAS: 6.8u, rcl:C-EUC1206
- removed CIN_1, CIN_2, CIN_3, COUT1_1, COUT1_2: 33u, rcl:C-USC1812
- removed COUT2_1, COUT2_2: 22u, rcl:C-USC1206
- removed D1, D2: MBRS140T3G, LAMS_lib:MBRS140T3G
- removed J1: PJ-070BH-SMT-TR, LAMS_lib:PJ-070BH-SMT-TR
- removed L2: MSS1260-682MLB, LAMS_lib:MSS1260-682MLB
- removed M1, M2, M3, M4: NVMFS5C468NL, LAMS_lib:NVMFS5C468NL
- removed RCS2: 20m, rcl:R-US_R1206
- removed ROSC: 46.4k, rcl:R-US_R0402
- removed R_CS1: 8.2m, rcl:R-US_R1206
- removed U1: MAX20034ATIS/VY+, LAMS_lib:MAX20034ATIS/VY+
- added BTN: LL3301BF065QJ, SamacSys_Parts:LL3301BF065QJ
- added C10: 4.7u, rcl:C-EUC1206
- added C11, C7, C8, C9: 100n, rcl:C-EUC1206
- added FERRITE_BEAD_1: BLA31AG221SN4D, SamacSys_Parts:BLA31AG221SN4D
- added J2: 1985920, SamacSys_Parts:1985920
- added JP4: (no value), pinhead:PINHD-1X9
- added R10: 1k, rcl:R-US_M1206
- added R5: 100k, rcl:R-US_M1206
- added R6, R7, R8: 10k, rcl:R-US_M1206
- added R9: 330, rcl:R-US_M1206
- added SD_CONN: GSD09002SEU, SamacSys_Parts:GSD09002SEU
- C1: value 4.7n -> 100n; device rcl:C-EUC0603 -> rcl:C-EUC1206
- C2: value 4.7p -> 10uF/10V; device rcl:C-EUC0402 -> rcl:C-EUC1206
- C3: value 4.7p -> 100n; device rcl:C-EUC0402 -> rcl:C-EUC1206
- C4: value 4.7n -> 10u; device rcl:C-EUC0603 -> rcl:C-EUC1206
- C5, C6: value 100n -> 10u; device rcl:C-EUC0603 -> rcl:C-EUC1206
- IC1: device LAMS_lib:ATSAME54N20A-AUT -> SamacSys_Parts:ATSAME54N20A-AUT
- L1: value SRP1238A-3R3M -> LQH31MN100J03L; device LAMS_lib:SRP1238A-3R3M -> SamacSys_Parts:LQH31MN100J03L
- R1: value 10.5k -> 100k; device rcl:R-US_R0402 -> rcl:R-US_M1206
- R2: value 10.2k -> 10k; device rcl:R-US_R0402 -> rcl:R-US_M1206
- R3, R4: value 51k -> 100k; device rcl:R-US_R0402 -> rcl:R-US_M1206
Connections:
- removed net BIAS: CBIAS.1, D1.A, D2.A, R3.1, R4.1, U1.BIAS, U1.FB1, U1.FB2, U1.FSYNC
- removed net BST1: C6.2, D2.K, U1.BST1
- removed net BST2: C5.2, D1.K, U1.BST2
- removed net COMP1: C2.1, R1.2, U1.COMP1
- removed net COMP2: C3.1, R2.2, U1.COMP2
- removed net CS1: L1.2, R_CS1.1, U1.CS1
- removed net CS2: L2.2, RCS2.1, U1.CS2
- removed net DH1: M2.G, U1.DH1
- removed net DH2: M1.G, U1.DH2
- removed net DL1: M4.G, U1.DL1
- removed net DL2: M3.G, U1.DL2
- removed net FOSC: ROSC.2, U1.FOSC
- removed net IN: CIN_1.1, CIN_2.1, CIN_3.1, J1.3, M1.D, M2.D, U1.EN1, U1.EN2, U1.IN
- removed net LIDAR_PWM: IC1.PB09
- removed net LIDAR_RX: IC1.PA05
- removed net LIDAR_TX: IC1.PA04
- removed net LX1: C6.1, L2.1, M2.S, M4.D, U1.LX1
- removed net LX2: C5.1, L1.1, M1.S, M3.D, U1.LX2
- removed net N$1: C1.1, R1.1
- removed net N$3: C4.1, R2.1
- removed net OUT1: COUT1_1.1, COUT1_2.1, R_CS1.2, U1.EXTVCC, U1.OUT1
- removed net OUT2: COUT2_1.1, COUT2_2.1, RCS2.2, U1.OUT2
- removed net PGOOD1: R3.2, U1.PGOOD1
- removed net PGOOD2: R4.2, U1.PGOOD2
- removed net SDDAT0: IC1.PB18
- removed net SDDAT1: IC1.PB19
- removed net SDDAT2: IC1.PB20
- removed net SDDAT3: IC1.PB21
- removed net SERVO_PWM: IC1.PA07
- removed net XIN1: IC1.PB22
- removed net XOUT1: IC1.PB23
- new net N$2: R2.1, SD_CONN.CMD
- new net N$4: BTN.NO_1, BTN.NO_2, R9.2
- new net SDCK: IC1.PB11, SD_CONN.CLK
- new net SDCMD: IC1.PA08
- new net SDDAT[0]: IC1.PA09, R3.1, SD_CONN.DAT0
- new net SDDAT[1]: IC1.PA10, R4.1, SD_CONN.DAT1
- new net SDDAT[2]: IC1.PA11, R5.1, SD_CONN.DAT2
- new net SDDAT[3]: IC1.PB10, R1.1, SD_CONN.DAT3
- new net VCC: C1.1, C2.1, J2.1, R1.2, R10.2, R2.2, R3.2, R4.2, R5.2, R6.2, R7.2, R8.2, SD_CONN.VDD
- net GND: now also BTN.COM_1, BTN.COM_2, C10.2, C11.2, C5.2, C6.2, C7.2, C8.2, C9.2, J2.2, SD_CONN.GND_1, SD_CONN.GND_2, SD_CONN.VSS1, SD_CONN.VSS2; no longer CBIAS.2, CIN_1.2, CIN_2.2, CIN_3.2, COUT1_1.2, COUT1_2.2, COUT2_1.2, COUT2_2.2, J1.1, J1.2, M3.S, M4.S, ROSC.1, U1.AGND, U1.EPAD, U1.PGND1, U1.PGND2
- net RESETN: now also C3.1, JP4.1, R8.1, R9.1
- net SDCD: now also IC1.PB12, R6.1, SD_CONN.CD; no longer IC1.PB16
- net SDWP: now also IC1.PB13, R7.1, SD_CONN.WRITE_PROTECT; no longer IC1.PB17
- net SWDCLK: now also JP4.3, R10.1
- net SWDIO: now also JP4.4
- net SWO: now also JP4.2
- net TRACECLK: now also JP4.9
- net TRACEDATA[0]: now also JP4.5
- net TRACEDATA[1]: now also JP4.6
- net TRACEDATA[2]: now also JP4.7
- net TRACEDATA[3]: now also JP4.8
- net VDDANA: now also C6.1, C8.1, FERRITE_BEAD_1.5, FERRITE_BEAD_1.6, FERRITE_BEAD_1.7, FERRITE_BEAD_1.8
- net VDDCORE: now also C10.1, C11.1, L1.1
- net VDDIO: now also C5.1, C9.1, FERRITE_BEAD_1.1, FERRITE_BEAD_1.2, FERRITE_BEAD_1.3, FERRITE_BEAD_1.4
- net VDDIOB: now also C4.1, C7.1
- net VSW: now also L1.2
Other:
- note added: "Pin headers optional"
- note added: "close to device (on every pin)"
- note removed: "*** Here I am assuming 3 as Vin *** *** check datasheet!!! ***"
- note removed: "1k"
- note removed: "ATSAME54 Pinout Usage"
- note removed: "Power / MAX20034"
