File: board_design/SAME54-board.sch (EAGLE design)
At the start: 32 parts, among them IC1 ATSAME54N20A-AUT, J1 PJ-070BH-SMT-TR, M1 NVMFS5C468NL, M2 NVMFS5C468NL, M3 NVMFS5C468NL, M4 NVMFS5C468NL, U1 MAX20034ATIS/VY+

Commit message: Updated schematic to include i/o, sd card, 12MHz clock
Parts:
- added C10, C11, C7, C8: 100n, rcl:C-EUC0603
- added C12, C13: 8p, rcl:C-EUC0603
- added C9: 10u, rcl:C-EUC0603
- added LIDAR: (no value), pinhead:PINHD-1X5
- added OSC1: CX3225CA12000D0KPSC1CX3225CA, LAMS_lib:CX3225CA12000D0KPSC1CX3225CA
- added PROG: (no value), pinhead:PINHD-1X10
- added R10, R11, R7, R9: 100k, rcl:R-US_R0603
- added R12, R13, R6, R8: 10k, rcl:R-US_R0603
- added R14: 1k, rcl:R-US_R0603
- added R5: 330, rcl:R-US_R0603
- added RESET_BTN: LL3301BF065QJ, LAMS_lib:LL3301BF065QJ
- added SD_CARD_CONN: GSD09002SEU, LAMS_lib:GSD09002SEU
- added SERVO: (no value), pinhead:PINHD-1X3
Connections:
- net IN renamed +9V
- removed net OUT1: COUT1_1.1, COUT1_2.1, R_CS1.2, U1.EXTVCC, U1.OUT1
- removed net OUT2: COUT2_1.1, COUT2_2.1, RCS2.2, U1.OUT2
- removed net VDDANA: IC1.VDDANA
- removed net VDDIO: IC1.VDDIO_1, IC1.VDDIO_2, IC1.VDDIO_3, IC1.VDDIO_4, IC1.VDDIO_5
- removed net VDDIOB: IC1.VDDIOB_1, IC1.VDDIOB_2
- removed net VSW: IC1.VSW
- new net +3V3: C10.1, C8.1, C9.1, COUT2_1.1, COUT2_2.1, IC1.VDDANA, IC1.VDDIOB_1, IC1.VDDIOB_2, IC1.VDDIO_1, IC1.VDDIO_2, IC1.VDDIO_3, IC1.VDDIO_4, IC1.VDDIO_5, R10.2, R11.2, R12.2, R13.2, R14.2, R6.2, R7.2, R8.2, R9.2, RCS2.2, SD_CARD_CONN.VDD, U1.OUT2
- new net +5V: COUT1_1.1, COUT1_2.1, LIDAR.1, R_CS1.2, SERVO.2, U1.EXTVCC, U1.OUT1
- new net N$4: R5.1, RESET_BTN.NO_1, RESET_BTN.NO_2
- new net SDCK: IC1.PA21, SD_CARD_CONN.CLK
- new net SDCMD: IC1.PA20, R8.1, SD_CARD_CONN.CMD
- net GND: now also C10.2, C11.2, C12.2, C13.2, C7.2, C8.2, C9.2, LIDAR.4, PROG.10, RESET_BTN.COM_1, RESET_BTN.COM_2, SD_CARD_CONN.GND_1, SD_CARD_CONN.GND_2, SD_CARD_CONN.VSS1, SD_CARD_CONN.VSS2, SERVO.3
- net LIDAR_PWM: now also LIDAR.5
- net LIDAR_RX: now also LIDAR.3
- net LIDAR_TX: now also LIDAR.2
- net RESETN: now also C7.1, PROG.1, R5.2, R6.1
- net SDCD: now also R12.1, SD_CARD_CONN.CD
- net SDDAT0: now also R9.1, SD_CARD_CONN.DAT0
- net SDDAT1: now also R10.1, SD_CARD_CONN.DAT1
- net SDDAT2: now also R11.1, SD_CARD_CONN.DAT2
- net SDDAT3: now also R7.1, SD_CARD_CONN.DAT3
- net SDWP: now also R13.1, SD_CARD_CONN.WRITE_PROTECT
- net SERVO_PWM: now also SERVO.1
- net SWDCLK: now also PROG.3, R14.1
- net SWDIO: now also PROG.4
- net SWO: now also PROG.2
- net TRACECLK: now also PROG.9
- net TRACEDATA[0]: now also PROG.5
- net TRACEDATA[1]: now also PROG.6
- net TRACEDATA[2]: now also PROG.7
- net TRACEDATA[3]: now also PROG.8
- net VDDCORE: now also C11.1
- net XIN1: now also C12.1, OSC1.1
- net XOUT1: now also C13.1, OSC1.3
Other:
- note added: "(internal voltage regulator output for monitoring)"
- note added: "SD Card Connections / 12MHz Clock / Pinheads / Reset Button"
- note added: "VDDANA"
- note added: "VDDIO"
- note added: "VDDIOB"
- note added: "decoupling capacitor"
- note added: "pull-up resistor"
- note removed: "1k"

Commit message: Finished custom SAME54 design. Ready to order
Parts:
- added C14: 4.7u, rcl:C-EUC0603
- added C15, C16: 100n, rcl:C-EUC0603
- renumbered R_CS1 to RCS1
Connections:
- net +3V3: now also C15.1, C16.1
- net +9V: now also J1.1; no longer J1.3
- net GND: now also C14.2, C15.2, C16.2, J1.3; no longer J1.1
- net VDDCORE: now also C14.1
Other:
- note added: "when no plug is inserted, 1 will be shorted to 3 1 - insertion detection 2 - sleeve 3 - tip"
- note removed: "*** Here I am assuming 3 as Vin *** *** check datasheet!!! ***"
- moved on the sheet: C11, J1

Commit message: Added diskio and fatfs middleware for file writing
Parts:
- added LED_RX, LED_STATUS, LED_TX: (no value), led:LEDCHIPLED_0603
- added R15: 10k, rcl:R-US_R0603
- added R16, R17, R18: (no value), rcl:R-US_R0603
- added START_BTN: LL3301BF065QJ, LAMS_lib:LL3301BF065QJ
- RCS1: value 8.2m -> 10m; device rcl:R-US_R1206 -> rcl:R-US_R0603
Connections:
- new net LED_STATUS: IC1.PA06, R16.2
- new net N$2: LED_STATUS.A, R16.1
- new net N$8: LED_RX.A, R17.1
- new net N$9: LED_TX.A, R18.1
- new net START_BTN: IC1.PA27, R15.2, START_BTN.COM_1, START_BTN.COM_2
- net +3V3: now also R17.2, R18.2, START_BTN.NO_1, START_BTN.NO_2
- net GND: now also LED_STATUS.C, R15.1
- net LIDAR_RX: now also LED_RX.C
- net LIDAR_TX: now also LED_TX.C
Other:
- note added: "SD Card Connections / 12MHz Clock / Pinheads / Buttons / LEDs"
- note added: "pull-down resistor"
- note removed: "SD Card Connections / 12MHz Clock / Pinheads / Reset Button"
- moved on the sheet: C12, C13, C7, C8, C9, LIDAR, OSC1, PROG, R10, R11, R12, R13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
